Commit message: -updated masses

File: ugv_description/urdf/ugv_core.xacro (robot description, xacro)
@@ -5,5 +5,5 @@
         <inertial>
             <origin xyz="5.607037937277861e-05 0.0 0.05002394672452172" rpy="0 0 0"/>
-            <mass value="52.779744190122"/>
+            <mass value="2"/>
             <inertia ixx="0.297294" iyy="0.389069" izz="0.598288" ixy="-0.0" iyz="0.0" ixz="-0.000163"/>
         </inertial>
@@ -25,5 +25,5 @@
         <inertial>
             <origin xyz="0.0 0.018500000000000072 -6.938893903907228e-18" rpy="0 0 0"/>
-            <mass value="1.45996093797625"/>
+            <mass value="0.0956"/>
             <inertia ixx="0.000751" iyy="0.001168" izz="0.000751" ixy="0.0" iyz="0.0" ixz="0.0"/>
         </inertial>
@@ -47,5 +47,5 @@
         <inertial>
             <origin xyz="-1.3877787807814457e-17 0.018500000000000072 -6.938893903907228e-18" rpy="0 0 0"/>
-            <mass value="1.45996093797625"/>
+            <mass value="0.0956"/>
             <inertia ixx="0.000751" iyy="0.001168" izz="0.000751" ixy="0.0" iyz="0.0" ixz="0.0"/>
         </inertial>
@@ -67,5 +67,5 @@
         <inertial>
             <origin xyz="-1.3877787807814457e-17 -0.01849999999999999 -6.938893903907228e-18" rpy="0 0 0"/>
-            <mass value="1.45996093797625"/>
+            <mass value="0.0956"/>
             <inertia ixx="0.000751" iyy="0.001168" izz="0.000751" ixy="0.0" iyz="0.0" ixz="0.0"/>
         </inertial>
@@ -89,5 +89,5 @@
         <inertial>
             <origin xyz="-1.1102230246251565e-15 -0.018500000000000072 -6.938893903907228e-18" rpy="0 0 0"/>
-            <mass value="1.45996093797625"/>
+            <mass value="0.0956"/>
             <inertia ixx="0.000751" iyy="0.001168" izz="0.000751" ixy="0.0" iyz="-0.0" ixz="-0.0"/>
         </inertial>

Commit message: -fixed mirrored axis!

File: ugv_description/urdf/ugv_core.xacro (robot description, xacro)
@@ -132,5 +132,5 @@
         <parent link="base_link"/>
         <child link="front_left_wheel"/>
-        <axis xyz="0.0 -1.0 0.0"/>
+        <axis xyz="0.0 1.0 0.0"/>
     </joint>
     <joint name="rear_left_wheel_joint" type="continuous">
@@ -150,5 +150,5 @@
         <parent link="base_link"/>
         <child link="front_right_wheel"/>
-        <axis xyz="0.0 -1.0 0.0"/>
+        <axis xyz="0.0 1.0 0.0"/>
     </joint>
     <joint name="lidar_link_joint" type="fixed">

Commit message: -new design

File: ugv_description/urdf/ugv_core.xacro (robot description, xacro)
@@ -4,7 +4,7 @@
     <link name="base_link">
         <inertial>
-            <origin xyz="5.607037937277861e-05 0.0 0.05002394672452172" rpy="0 0 0"/>
+            <origin xyz="0.0 1.7728771913886266e-17 0.10999933880977349" rpy="0 0 0"/>
             <mass value="2"/>
-            <inertia ixx="0.297294" iyy="0.389069" izz="0.598288" ixy="-0.0" iyz="0.0" ixz="-0.000163"/>
+            <inertia ixx="0.966516" iyy="1.898649" izz="2.169279" ixy="0.0" iyz="0.0" ixz="0.0"/>
         </inertial>
         <visual>
@@ -24,21 +24,19 @@
     <link name="front_left_wheel">
         <inertial>
-            <origin xyz="0.0 0.018500000000000072 -6.938893903907228e-18" rpy="0 0 0"/>
+            <origin xyz="0.0 0.020000000000000018 -6.938893903907228e-18" rpy="0 0 0"/>
             <mass value="0.0956"/>
-            <inertia ixx="0.000751" iyy="0.001168" izz="0.000751" ixy="0.0" iyz="0.0" ixz="0.0"/>
+            <inertia ixx="0.000842" iyy="0.001263" izz="0.000842" ixy="-0.0" iyz="-0.0" ixz="-0.0"/>
         </inertial>
         <visual>
-            <origin xyz="-0.09841 -0.125 -0.02" rpy="0 0 0"/>
+            <origin xyz="-0.13672 -0.122 -0.0409" rpy="0 0 0"/>
             <geometry>
-                <mesh filename="file://$(find ugv_description)/meshes/front_left_wheel.stl"
-                      scale="0.001 0.001 0.001"/>
+                <mesh filename="file://$(find ugv_description)/meshes/front_left_wheel.stl" scale="0.001 0.001 0.001"/>
             </geometry>
             <material name="silver"/>
         </visual>
         <collision>
-            <origin xyz="-0.09841 -0.125 -0.02" rpy="0 0 0"/>
+            <origin xyz="-0.13672 -0.122 -0.0409" rpy="0 0 0"/>
             <geometry>
-                <mesh filename="file://$(find ugv_description)/meshes/front_left_wheel.stl"
-                      scale="0.001 0.001 0.001"/>
+                <mesh filename="file://$(find ugv_description)/meshes/front_left_wheel.stl" scale="0.001 0.001 0.001"/>
             </geometry>
         </collision>
@@ -46,10 +44,10 @@
     <link name="rear_left_wheel">
         <inertial>
-            <origin xyz="-1.3877787807814457e-17 0.018500000000000072 -6.938893903907228e-18" rpy="0 0 0"/>
+            <origin xyz="-2.7755575615628914e-17 0.020000000000000018 -6.938893903907228e-18" rpy="0 0 0"/>
             <mass value="0.0956"/>
-            <inertia ixx="0.000751" iyy="0.001168" izz="0.000751" ixy="0.0" iyz="0.0" ixz="0.0"/>
+            <inertia ixx="0.000842" iyy="0.001263" izz="0.000842" ixy="-0.0" iyz="-0.0" ixz="0.0"/>
         </inertial>
         <visual>
-            <origin xyz="0.09841 -0.125 -0.02" rpy="0 0 0"/>
+            <origin xyz="0.13672 -0.122 -0.0409" rpy="0 0 0"/>
             <geometry>
                 <mesh filename="file://$(find ugv_description)/meshes/rear_left_wheel.stl" scale="0.001 0.001 0.001"/>
@@ -58,5 +56,5 @@
         </visual>
         <collision>
-            <origin xyz="0.09841 -0.125 -0.02" rpy="0 0 0"/>
+            <origin xyz="0.13672 -0.122 -0.0409" rpy="0 0 0"/>
             <geometry>
                 <mesh filename="file://$(find ugv_description)/meshes/rear_left_wheel.stl" scale="0.001 0.001 0.001"/>
@@ -66,21 +64,19 @@
     <link name="rear_right_wheel">
         <inertial>
-            <origin xyz="-1.3877787807814457e-17 -0.01849999999999999 -6.938893903907228e-18" rpy="0 0 0"/>
+            <origin xyz="0.0 -0.020000000000000018 0.0" rpy="0 0 0"/>
             <mass value="0.0956"/>
-            <inertia ixx="0.000751" iyy="0.001168" izz="0.000751" ixy="0.0" iyz="0.0" ixz="0.0"/>
+            <inertia ixx="0.000842" iyy="0.001263" izz="0.000842" ixy="-0.0" iyz="0.0" ixz="0.0"/>
         </inertial>
         <visual>
-            <origin xyz="0.09841 0.125 -0.02" rpy="0 0 0"/>
+            <origin xyz="0.13672 0.122 -0.0409" rpy="0 0 0"/>
             <geometry>
-                <mesh filename="file://$(find ugv_description)/meshes/rear_right_wheel.stl"
-                      scale="0.001 0.001 0.001"/>
+                <mesh filename="file://$(find ugv_description)/meshes/rear_right_wheel.stl" scale="0.001 0.001 0.001"/>
             </geometry>
             <material name="silver"/>
         </visual>
         <collision>
-            <origin xyz="0.09841 0.125 -0.02" rpy="0 0 0"/>
+            <origin xyz="0.13672 0.122 -0.0409" rpy="0 0 0"/>
             <geometry>
-                <mesh filename="file://$(find ugv_description)/meshes/rear_right_wheel.stl"
-                      scale="0.001 0.001 0.001"/>
+                <mesh filename="file://$(find ugv_description)/meshes/rear_right_wheel.stl" scale="0.001 0.001 0.001"/>
             </geometry>
         </collision>
@@ -88,21 +84,19 @@
     <link name="front_right_wheel">
         <inertial>
-            <origin xyz="-1.1102230246251565e-15 -0.018500000000000072 -6.938893903907228e-18" rpy="0 0 0"/>
+            <origin xyz="0.0 -0.020000000000000018 0.0" rpy="0 0 0"/>
             <mass value="0.0956"/>
-            <inertia ixx="0.000751" iyy="0.001168" izz="0.000751" ixy="0.0" iyz="-0.0" ixz="-0.0"/>
+            <inertia ixx="0.000842" iyy="0.001263" izz="0.000842" ixy="-0.0" iyz="0.0" ixz="0.0"/>
         </inertial>
         <visual>
-            <origin xyz="-0.09841 0.125 -0.02" rpy="0 0 0"/>
+            <origin xyz="-0.13672 0.122 -0.0409" rpy="0 0 0"/>
             <geometry>
-                <mesh filename="file://$(find ugv_description)/meshes/front_right_wheel.stl"
-                      scale="0.001 0.001 0.001"/>
+                <mesh filename="file://$(find ugv_description)/meshes/front_right_wheel.stl" scale="0.001 0.001 0.001"/>
             </geometry>
             <material name="silver"/>
         </visual>
         <collision>
-            <origin xyz="-0.09841 0.125 -0.02" rpy="0 0 0"/>
+            <origin xyz="-0.13672 0.122 -0.0409" rpy="0 0 0"/>
             <geometry>
-                <mesh filename="file://$(find ugv_description)/meshes/front_right_wheel.stl"
-                      scale="0.001 0.001 0.001"/>
+                <mesh filename="file://$(find ugv_description)/meshes/front_right_wheel.stl" scale="0.001 0.001 0.001"/>
             </geometry>
         </collision>
@@ -110,10 +104,10 @@
     <link name="lidar_link">
         <inertial>
-            <origin xyz="0.0 7.237528875152536e-18 0.009999999999999995" rpy="0 0 0"/>
-            <mass value="0.3082687791334984"/>
-            <inertia ixx="5.8e-05" iyy="5.8e-05" izz="9.6e-05" ixy="0.0" iyz="-0.0" ixz="0.0"/>
+            <origin xyz="-0.027115069985041318 3.5226945429821856e-06 -0.0020552178870618665" rpy="0 0 0"/>
+            <mass value="0.7886321015037847"/>
+            <inertia ixx="0.000269" iyy="0.000272" izz="0.000333" ixy="0.0" iyz="0.0" ixz="-1e-06"/>
         </inertial>
         <visual>
-            <origin xyz="-0.12 -0.0 -0.11" rpy="0 0 0"/>
+            <origin xyz="-0.19 -0.0 -0.22" rpy="0 0 0"/>
             <geometry>
                 <mesh filename="file://$(find ugv_description)/meshes/lidar_link.stl" scale="0.001 0.001 0.001"/>
@@ -122,5 +116,5 @@
         </visual>
         <collision>
-            <origin xyz="-0.12 -0.0 -0.11" rpy="0 0 0"/>
+            <origin xyz="-0.19 -0.0 -0.22" rpy="0 0 0"/>
             <geometry>
                 <mesh filename="file://$(find ugv_description)/meshes/lidar_link.stl" scale="0.001 0.001 0.001"/>
@@ -129,5 +123,5 @@
     </link>
     <joint name="front_left_wheel_joint" type="continuous">
-        <origin xyz="0.09841 0.125 0.02" rpy="0 0 0"/>
+        <origin xyz="0.13672 0.122 0.0409" rpy="0 0 0"/>
         <parent link="base_link"/>
         <child link="front_left_wheel"/>
@@ -135,5 +129,5 @@
     </joint>
     <joint name="rear_left_wheel_joint" type="continuous">
-        <origin xyz="-0.09841 0.125 0.02" rpy="0 0 0"/>
+        <origin xyz="-0.13672 0.122 0.0409" rpy="0 0 0"/>
         <parent link="base_link"/>
         <child link="rear_left_wheel"/>
@@ -141,5 +135,5 @@
     </joint>
     <joint name="rear_right_wheel_joint" type="continuous">
-        <origin xyz="-0.09841 -0.125 0.02" rpy="0 0 0"/>
+        <origin xyz="-0.13672 -0.122 0.0409" rpy="0 0 0"/>
         <parent link="base_link"/>
         <child link="rear_right_wheel"/>
@@ -147,5 +141,5 @@
     </joint>
     <joint name="front_right_wheel_joint" type="continuous">
-        <origin xyz="0.09841 -0.125 0.02" rpy="0 0 0"/>
+        <origin xyz="0.13672 -0.122 0.0409" rpy="0 0 0"/>
         <parent link="base_link"/>
         <child link="front_right_wheel"/>
@@ -153,5 +147,5 @@
     </joint>
     <joint name="lidar_link_joint" type="fixed">
-        <origin xyz="0.12 0.0 0.11" rpy="0 0 0"/>
+        <origin xyz="0.19 0.0 0.22" rpy="0 0 0"/>
         <parent link="base_link"/>
         <child link="lidar_link"/>

Commit message: inertia macros

File: ugv_description/urdf/ugv_core.xacro (robot description, xacro)
@@ -2,9 +2,23 @@
 <robot name="ugv" xmlns:xacro="http://www.ros.org/wiki/xacro">
     <xacro:include filename="$(find ugv_description)/urdf/materials.xacro"/>
+    <xacro:property name="base_link_mass" value="2"/>
+    <xacro:property name="wheel_mass" value="0.0956"/>
+    <xacro:property name="wheel_radius" value="0.04"/>
+    <xacro:property name="wheel_height" value="0.04"/>
+    <xacro:macro name="box_inertia" params="m x y z">
+        <inertia  ixx="${m*(y*y+z*z)/12}" ixy = "0" ixz = "0"
+                  iyy="${m*(x*x+z*z)/12}" iyz = "0"
+                  izz="${m*(x*x+z*z)/12}" />
+    </xacro:macro>
+    <xacro:macro name="cylinder_inertia" params="m r h">
+      <inertia  ixx="${m*(3*r*r+h*h)/12}" ixy = "0" ixz = "0"
+                  iyy="${m*(3*r*r+h*h)/12}" iyz = "0"
+                  izz="${m*r*r/2}" />
+      </xacro:macro>
     <link name="base_link">
         <inertial>
-            <origin xyz="0.0 1.7728771913886266e-17 0.10999933880977349" rpy="0 0 0"/>
-            <mass value="2"/>
-            <inertia ixx="0.966516" iyy="1.898649" izz="2.169279" ixy="0.0" iyz="0.0" ixz="0.0"/>
+            <origin xyz="0 0 0" rpy="0 0 0"/>
+            <mass value="${base_link_mass}"/>
+            <xacro:box_inertia m="${base_link_mass}" x=".38" y=".24" z=".18" />
         </inertial>
         <visual>
@@ -25,6 +39,6 @@
         <inertial>
             <origin xyz="0.0 0.020000000000000018 -6.938893903907228e-18" rpy="0 0 0"/>
-            <mass value="0.0956"/>
-            <inertia ixx="0.000842" iyy="0.001263" izz="0.000842" ixy="-0.0" iyz="-0.0" ixz="-0.0"/>
+            <mass value="${wheel_mass}"/>
+            <xacro:cylinder_inertia m="${wheel_mass}" r="${wheel_radius}" h="${wheel_height}" />
         </inertial>
         <visual>
@@ -45,6 +59,6 @@
         <inertial>
             <origin xyz="-2.7755575615628914e-17 0.020000000000000018 -6.938893903907228e-18" rpy="0 0 0"/>
-            <mass value="0.0956"/>
-            <inertia ixx="0.000842" iyy="0.001263" izz="0.000842" ixy="-0.0" iyz="-0.0" ixz="0.0"/>
+            <mass value="${wheel_mass}"/>
+            <xacro:cylinder_inertia m="${wheel_mass}" r="${wheel_radius}" h="${wheel_height}" />
         </inertial>
         <visual>
@@ -65,6 +79,6 @@
         <inertial>
             <origin xyz="0.0 -0.020000000000000018 0.0" rpy="0 0 0"/>
-            <mass value="0.0956"/>
-            <inertia ixx="0.000842" iyy="0.001263" izz="0.000842" ixy="-0.0" iyz="0.0" ixz="0.0"/>
+            <mass value="${wheel_mass}"/>
+           <xacro:cylinder_inertia m="${wheel_mass}" r="${wheel_radius}" h="${wheel_height}" />
         </inertial>
         <visual>
@@ -85,7 +99,7 @@
         <inertial>
             <origin xyz="0.0 -0.020000000000000018 0.0" rpy="0 0 0"/>
-            <mass value="0.0956"/>
-            <inertia ixx="0.000842" iyy="0.001263" izz="0.000842" ixy="-0.0" iyz="0.0" ixz="0.0"/>
-        </inertial>
+            <mass value="${wheel_mass}"/>
+             <xacro:cylinder_inertia m="${wheel_mass}" r="${wheel_radius}" h="${wheel_height}" />
+       </inertial>
         <visual>
             <origin xyz="-0.13672 0.122 -0.0409" rpy="0 0 0"/>
@@ -106,6 +120,6 @@
             <origin xyz="-0.027115069985041318 3.5226945429821856e-06 -0.0020552178870618665" rpy="0 0 0"/>
             <mass value="0.7886321015037847"/>
-            <inertia ixx="0.000269" iyy="0.000272" izz="0.000333" ixy="0.0" iyz="0.0" ixz="-1e-06"/>
-        </inertial>
+            <xacro:cylinder_inertia m="${wheel_mass}" r="${wheel_radius}" h="${wheel_height}" />
+     </inertial>
         <visual>
             <origin xyz="-0.19 -0.0 -0.22" rpy="0 0 0"/>

Commit message: -passing gazebo world to control launch

File: ugv_description/urdf/ugv_core.xacro (robot description, xacro)
@@ -2,23 +2,9 @@
 <robot name="ugv" xmlns:xacro="http://www.ros.org/wiki/xacro">
     <xacro:include filename="$(find ugv_description)/urdf/materials.xacro"/>
-    <xacro:property name="base_link_mass" value="2"/>
-    <xacro:property name="wheel_mass" value="0.0956"/>
-    <xacro:property name="wheel_radius" value="0.04"/>
-    <xacro:property name="wheel_height" value="0.04"/>
-    <xacro:macro name="box_inertia" params="m x y z">
-        <inertia  ixx="${m*(y*y+z*z)/12}" ixy = "0" ixz = "0"
-                  iyy="${m*(x*x+z*z)/12}" iyz = "0"
-                  izz="${m*(x*x+z*z)/12}" />
-    </xacro:macro>
-    <xacro:macro name="cylinder_inertia" params="m r h">
-      <inertia  ixx="${m*(3*r*r+h*h)/12}" ixy = "0" ixz = "0"
-                  iyy="${m*(3*r*r+h*h)/12}" iyz = "0"
-                  izz="${m*r*r/2}" />
-      </xacro:macro>
     <link name="base_link">
         <inertial>
-            <origin xyz="0 0 0" rpy="0 0 0"/>
-            <mass value="${base_link_mass}"/>
-            <xacro:box_inertia m="${base_link_mass}" x=".38" y=".24" z=".18" />
+            <origin xyz="0.0 1.7728771913886266e-17 0.10999933880977349" rpy="0 0 0"/>
+            <mass value="2"/>
+            <inertia ixx="0.966516" iyy="1.898649" izz="2.169279" ixy="0.0" iyz="0.0" ixz="0.0"/>
         </inertial>
         <visual>
@@ -39,6 +25,6 @@
         <inertial>
             <origin xyz="0.0 0.020000000000000018 -6.938893903907228e-18" rpy="0 0 0"/>
-            <mass value="${wheel_mass}"/>
-            <xacro:cylinder_inertia m="${wheel_mass}" r="${wheel_radius}" h="${wheel_height}" />
+            <mass value="0.0956"/>
+            <inertia ixx="0.000842" iyy="0.001263" izz="0.000842" ixy="-0.0" iyz="-0.0" ixz="-0.0"/>
         </inertial>
         <visual>
@@ -59,6 +45,6 @@
         <inertial>
             <origin xyz="-2.7755575615628914e-17 0.020000000000000018 -6.938893903907228e-18" rpy="0 0 0"/>
-            <mass value="${wheel_mass}"/>
-            <xacro:cylinder_inertia m="${wheel_mass}" r="${wheel_radius}" h="${wheel_height}" />
+            <mass value="0.0956"/>
+            <inertia ixx="0.000842" iyy="0.001263" izz="0.000842" ixy="-0.0" iyz="-0.0" ixz="0.0"/>
         </inertial>
         <visual>
@@ -79,6 +65,6 @@
         <inertial>
             <origin xyz="0.0 -0.020000000000000018 0.0" rpy="0 0 0"/>
-            <mass value="${wheel_mass}"/>
-           <xacro:cylinder_inertia m="${wheel_mass}" r="${wheel_radius}" h="${wheel_height}" />
+            <mass value="0.0956"/>
+            <inertia ixx="0.000842" iyy="0.001263" izz="0.000842" ixy="-0.0" iyz="0.0" ixz="0.0"/>
         </inertial>
         <visual>
@@ -99,7 +85,7 @@
         <inertial>
             <origin xyz="0.0 -0.020000000000000018 0.0" rpy="0 0 0"/>
-            <mass value="${wheel_mass}"/>
-             <xacro:cylinder_inertia m="${wheel_mass}" r="${wheel_radius}" h="${wheel_height}" />
-       </inertial>
+            <mass value="0.0956"/>
+            <inertia ixx="0.000842" iyy="0.001263" izz="0.000842" ixy="-0.0" iyz="0.0" ixz="0.0"/>
+        </inertial>
         <visual>
             <origin xyz="-0.13672 0.122 -0.0409" rpy="0 0 0"/>
@@ -120,6 +106,6 @@
             <origin xyz="-0.027115069985041318 3.5226945429821856e-06 -0.0020552178870618665" rpy="0 0 0"/>
             <mass value="0.7886321015037847"/>
-            <xacro:cylinder_inertia m="${wheel_mass}" r="${wheel_radius}" h="${wheel_height}" />
-     </inertial>
+            <inertia ixx="0.000269" iyy="0.000272" izz="0.000333" ixy="0.0" iyz="0.0" ixz="-1e-06"/>
+        </inertial>
         <visual>
             <origin xyz="-0.19 -0.0 -0.22" rpy="0 0 0"/>
