Commit message: -new design

File: ugv_description/urdf/ugv_core.xacro (robot description, xacro)
@@ -4,7 +4,7 @@
     <link name="base_link">
         <inertial>
-            <origin xyz="0.0 1.7728771913886266e-17 0.10999933880977349" rpy="0 0 0"/>
-            <mass value="2"/>
-            <inertia ixx="0.966516" iyy="1.898649" izz="2.169279" ixy="0.0" iyz="0.0" ixz="0.0"/>
+            <origin xyz="-0.001286687391743976 5.852613032120841e-06 0.0774595073842539" rpy="0 0 0"/>
+            <mass value="1.8659797599914978"/>
+            <inertia ixx="0.018308" iyy="0.036464" izz="0.054285" ixy="0.0" iyz="0.0" ixz="-2.4e-05"/>
         </inertial>
         <visual>
@@ -24,10 +24,10 @@
     <link name="front_left_wheel">
         <inertial>
-            <origin xyz="0.0 0.020000000000000018 -6.938893903907228e-18" rpy="0 0 0"/>
-            <mass value="0.0956"/>
-            <inertia ixx="0.000842" iyy="0.001263" izz="0.000842" ixy="-0.0" iyz="-0.0" ixz="-0.0"/>
+            <origin xyz="1.2352069053700454e-07 0.01999978800742533 2.9802318252114546e-10" rpy="0 0 0"/>
+            <mass value="1.578336149163512"/>
+            <inertia ixx="0.000842" iyy="0.001263" izz="0.000842" ixy="0.0" iyz="0.0" ixz="-0.0"/>
         </inertial>
         <visual>
-            <origin xyz="-0.13672 -0.122 -0.0409" rpy="0 0 0"/>
+            <origin xyz="-0.143415 -0.123006 -0.0425" rpy="0 0 0"/>
             <geometry>
                 <mesh filename="file://$(find ugv_description)/meshes/front_left_wheel.stl" scale="0.001 0.001 0.001"/>
@@ -36,5 +36,5 @@
         </visual>
         <collision>
-            <origin xyz="-0.13672 -0.122 -0.0409" rpy="0 0 0"/>
+            <origin xyz="-0.143415 -0.123006 -0.0425" rpy="0 0 0"/>
             <geometry>
                 <mesh filename="file://$(find ugv_description)/meshes/front_left_wheel.stl" scale="0.001 0.001 0.001"/>
@@ -44,10 +44,10 @@
     <link name="rear_left_wheel">
         <inertial>
-            <origin xyz="-2.7755575615628914e-17 0.020000000000000018 -6.938893903907228e-18" rpy="0 0 0"/>
-            <mass value="0.0956"/>
-            <inertia ixx="0.000842" iyy="0.001263" izz="0.000842" ixy="-0.0" iyz="-0.0" ixz="0.0"/>
+            <origin xyz="1.235206903704711e-07 0.019999788007424774 2.9802318252114546e-10" rpy="0 0 0"/>
+            <mass value="1.578336149163512"/>
+            <inertia ixx="0.000842" iyy="0.001263" izz="0.000842" ixy="0.0" iyz="-0.0" ixz="0.0"/>
         </inertial>
         <visual>
-            <origin xyz="0.13672 -0.122 -0.0409" rpy="0 0 0"/>
+            <origin xyz="0.147785 -0.123006 -0.0425" rpy="0 0 0"/>
             <geometry>
                 <mesh filename="file://$(find ugv_description)/meshes/rear_left_wheel.stl" scale="0.001 0.001 0.001"/>
@@ -56,5 +56,5 @@
         </visual>
         <collision>
-            <origin xyz="0.13672 -0.122 -0.0409" rpy="0 0 0"/>
+            <origin xyz="0.147785 -0.123006 -0.0425" rpy="0 0 0"/>
             <geometry>
                 <mesh filename="file://$(find ugv_description)/meshes/rear_left_wheel.stl" scale="0.001 0.001 0.001"/>
@@ -62,12 +62,32 @@
         </collision>
     </link>
+    <link name="front_right_wheel">
+        <inertial>
+            <origin xyz="1.235206901206709e-07 -0.020000211992574804 2.9802321027672107e-10" rpy="0 0 0"/>
+            <mass value="1.578336149163512"/>
+            <inertia ixx="0.000842" iyy="0.001263" izz="0.000842" ixy="0.0" iyz="0.0" ixz="0.0"/>
+        </inertial>
+        <visual>
+            <origin xyz="-0.143415 0.122994 -0.0425" rpy="0 0 0"/>
+            <geometry>
+                <mesh filename="file://$(find ugv_description)/meshes/front_right_wheel.stl" scale="0.001 0.001 0.001"/>
+            </geometry>
+            <material name="silver"/>
+        </visual>
+        <collision>
+            <origin xyz="-0.143415 0.122994 -0.0425" rpy="0 0 0"/>
+            <geometry>
+                <mesh filename="file://$(find ugv_description)/meshes/front_right_wheel.stl" scale="0.001 0.001 0.001"/>
+            </geometry>
+        </collision>
+    </link>
     <link name="rear_right_wheel">
         <inertial>
-            <origin xyz="0.0 -0.020000000000000018 0.0" rpy="0 0 0"/>
-            <mass value="0.0956"/>
-            <inertia ixx="0.000842" iyy="0.001263" izz="0.000842" ixy="-0.0" iyz="0.0" ixz="0.0"/>
+            <origin xyz="1.2352069095333817e-07 -0.020000211992574915 2.9802314782667594e-10" rpy="0 0 0"/>
+            <mass value="1.578336149163512"/>
+            <inertia ixx="0.000842" iyy="0.001263" izz="0.000842" ixy="0.0" iyz="0.0" ixz="0.0"/>
         </inertial>
         <visual>
-            <origin xyz="0.13672 0.122 -0.0409" rpy="0 0 0"/>
+            <origin xyz="0.147785 0.122994 -0.0425" rpy="0 0 0"/>
             <geometry>
                 <mesh filename="file://$(find ugv_description)/meshes/rear_right_wheel.stl" scale="0.001 0.001 0.001"/>
@@ -76,5 +96,5 @@
         </visual>
         <collision>
-            <origin xyz="0.13672 0.122 -0.0409" rpy="0 0 0"/>
+            <origin xyz="0.147785 0.122994 -0.0425" rpy="0 0 0"/>
             <geometry>
                 <mesh filename="file://$(find ugv_description)/meshes/rear_right_wheel.stl" scale="0.001 0.001 0.001"/>
@@ -82,32 +102,12 @@
         </collision>
     </link>
-    <link name="front_right_wheel">
-        <inertial>
-            <origin xyz="0.0 -0.020000000000000018 0.0" rpy="0 0 0"/>
-            <mass value="0.0956"/>
-            <inertia ixx="0.000842" iyy="0.001263" izz="0.000842" ixy="-0.0" iyz="0.0" ixz="0.0"/>
-        </inertial>
-        <visual>
-            <origin xyz="-0.13672 0.122 -0.0409" rpy="0 0 0"/>
-            <geometry>
-                <mesh filename="file://$(find ugv_description)/meshes/front_right_wheel.stl" scale="0.001 0.001 0.001"/>
-            </geometry>
-            <material name="silver"/>
-        </visual>
-        <collision>
-            <origin xyz="-0.13672 0.122 -0.0409" rpy="0 0 0"/>
-            <geometry>
-                <mesh filename="file://$(find ugv_description)/meshes/front_right_wheel.stl" scale="0.001 0.001 0.001"/>
-            </geometry>
-        </collision>
-    </link>
     <link name="lidar_link">
         <inertial>
-            <origin xyz="-0.027115069985041318 3.5226945429821856e-06 -0.0020552178870618665" rpy="0 0 0"/>
+            <origin xyz="-0.00011494677727549862 3.3107019681208537e-06 0.017944782112938054" rpy="0 0 0"/>
             <mass value="0.7886321015037847"/>
             <inertia ixx="0.000269" iyy="0.000272" izz="0.000333" ixy="0.0" iyz="0.0" ixz="-1e-06"/>
         </inertial>
         <visual>
-            <origin xyz="-0.19 -0.0 -0.22" rpy="0 0 0"/>
+            <origin xyz="-0.186715 -6e-06 -0.091" rpy="0 0 0"/>
             <geometry>
                 <mesh filename="file://$(find ugv_description)/meshes/lidar_link.stl" scale="0.001 0.001 0.001"/>
@@ -116,5 +116,5 @@
         </visual>
         <collision>
-            <origin xyz="-0.19 -0.0 -0.22" rpy="0 0 0"/>
+            <origin xyz="-0.186715 -6e-06 -0.091" rpy="0 0 0"/>
             <geometry>
                 <mesh filename="file://$(find ugv_description)/meshes/lidar_link.stl" scale="0.001 0.001 0.001"/>
@@ -123,29 +123,29 @@
     </link>
     <joint name="front_left_wheel_joint" type="continuous">
-        <origin xyz="0.13672 0.122 0.0409" rpy="0 0 0"/>
+        <origin xyz="0.143415 0.123006 0.0425" rpy="0 0 0"/>
         <parent link="base_link"/>
         <child link="front_left_wheel"/>
-        <axis xyz="0.0 1.0 0.0"/>
+        <axis xyz="0.0 -1.0 0.0"/>
     </joint>
     <joint name="rear_left_wheel_joint" type="continuous">
-        <origin xyz="-0.13672 0.122 0.0409" rpy="0 0 0"/>
+        <origin xyz="-0.147785 0.123006 0.0425" rpy="0 0 0"/>
         <parent link="base_link"/>
         <child link="rear_left_wheel"/>
-        <axis xyz="0.0 1.0 0.0"/>
+        <axis xyz="0.0 -1.0 0.0"/>
+    </joint>
+    <joint name="front_right_wheel_joint" type="continuous">
+        <origin xyz="0.143415 -0.122994 0.0425" rpy="0 0 0"/>
+        <parent link="base_link"/>
+        <child link="front_right_wheel"/>
+        <axis xyz="-0.0 1.0 -0.0"/>
     </joint>
     <joint name="rear_right_wheel_joint" type="continuous">
-        <origin xyz="-0.13672 -0.122 0.0409" rpy="0 0 0"/>
+        <origin xyz="-0.147785 -0.122994 0.0425" rpy="0 0 0"/>
         <parent link="base_link"/>
         <child link="rear_right_wheel"/>
-        <axis xyz="0.0 1.0 0.0"/>
-    </joint>
-    <joint name="front_right_wheel_joint" type="continuous">
-        <origin xyz="0.13672 -0.122 0.0409" rpy="0 0 0"/>
-        <parent link="base_link"/>
-        <child link="front_right_wheel"/>
-        <axis xyz="0.0 1.0 0.0"/>
+        <axis xyz="-0.0 1.0 -0.0"/>
     </joint>
     <joint name="lidar_link_joint" type="fixed">
-        <origin xyz="0.19 0.0 0.22" rpy="0 0 0"/>
+        <origin xyz="0.186715 6e-06 0.091" rpy="0 0 0"/>
         <parent link="base_link"/>
         <child link="lidar_link"/>

Commit message: -new design

File: ugv_description/urdf/ugv_core.xacro (robot description, xacro)
@@ -4,7 +4,7 @@
     <link name="base_link">
         <inertial>
-            <origin xyz="-0.001286687391743976 5.852613032120841e-06 0.0774595073842539" rpy="0 0 0"/>
-            <mass value="1.8659797599914978"/>
-            <inertia ixx="0.018308" iyy="0.036464" izz="0.054285" ixy="0.0" iyz="0.0" ixz="-2.4e-05"/>
+            <origin xyz="0.25539221363619424 -0.008191452128420306 0.07740258559841702" rpy="0 0 0"/>
+            <mass value="1.8582255296411472"/>
+            <inertia ixx="0.018307" iyy="0.036178" izz="0.054" ixy="-3e-06" iyz="-0.0" ixz="-5e-06"/>
         </inertial>
         <visual>
@@ -22,41 +22,21 @@
         </collision>
     </link>
-    <link name="front_left_wheel">
+    <link name="lidar_link">
         <inertial>
-            <origin xyz="1.2352069053700454e-07 0.01999978800742533 2.9802318252114546e-10" rpy="0 0 0"/>
-            <mass value="1.578336149163512"/>
-            <inertia ixx="0.000842" iyy="0.001263" izz="0.000842" ixy="0.0" iyz="0.0" ixz="-0.0"/>
+            <origin xyz="-0.0001155547326693318 3.2715051849067412e-06 0.01794478211293804" rpy="0 0 0"/>
+            <mass value="0.7886321015037847"/>
+            <inertia ixx="0.000269" iyy="0.000272" izz="0.000333" ixy="0.0" iyz="0.0" ixz="-1e-06"/>
         </inertial>
         <visual>
-            <origin xyz="-0.143415 -0.123006 -0.0425" rpy="0 0 0"/>
+            <origin xyz="-0.43536 6e-05 -0.091" rpy="0 0 0"/>
             <geometry>
-                <mesh filename="file://$(find ugv_description)/meshes/front_left_wheel.stl" scale="0.001 0.001 0.001"/>
+                <mesh filename="file://$(find ugv_description)/meshes/lidar_link.stl" scale="0.001 0.001 0.001"/>
             </geometry>
             <material name="silver"/>
         </visual>
         <collision>
-            <origin xyz="-0.143415 -0.123006 -0.0425" rpy="0 0 0"/>
+            <origin xyz="-0.43536 6e-05 -0.091" rpy="0 0 0"/>
             <geometry>
-                <mesh filename="file://$(find ugv_description)/meshes/front_left_wheel.stl" scale="0.001 0.001 0.001"/>
-            </geometry>
-        </collision>
-    </link>
-    <link name="rear_left_wheel">
-        <inertial>
-            <origin xyz="1.235206903704711e-07 0.019999788007424774 2.9802318252114546e-10" rpy="0 0 0"/>
-            <mass value="1.578336149163512"/>
-            <inertia ixx="0.000842" iyy="0.001263" izz="0.000842" ixy="0.0" iyz="-0.0" ixz="0.0"/>
-        </inertial>
-        <visual>
-            <origin xyz="0.147785 -0.123006 -0.0425" rpy="0 0 0"/>
-            <geometry>
-                <mesh filename="file://$(find ugv_description)/meshes/rear_left_wheel.stl" scale="0.001 0.001 0.001"/>
-            </geometry>
-            <material name="silver"/>
-        </visual>
-        <collision>
-            <origin xyz="0.147785 -0.123006 -0.0425" rpy="0 0 0"/>
-            <geometry>
-                <mesh filename="file://$(find ugv_description)/meshes/rear_left_wheel.stl" scale="0.001 0.001 0.001"/>
+                <mesh filename="file://$(find ugv_description)/meshes/lidar_link.stl" scale="0.001 0.001 0.001"/>
             </geometry>
         </collision>
@@ -64,10 +44,10 @@
     <link name="front_right_wheel">
         <inertial>
-            <origin xyz="1.235206901206709e-07 -0.020000211992574804 2.9802321027672107e-10" rpy="0 0 0"/>
-            <mass value="1.578336149163512"/>
-            <inertia ixx="0.000842" iyy="0.001263" izz="0.000842" ixy="0.0" iyz="0.0" ixz="0.0"/>
+            <origin xyz="-3.129242420740752e-10 -0.018799999999999678 2.9802320333782717e-10" rpy="0 0 0"/>
+            <mass value="1.4688367113110694"/>
+            <inertia ixx="0.000755" iyy="0.001163" izz="0.000755" ixy="0.0" iyz="0.0" ixz="-0.0"/>
         </inertial>
         <visual>
-            <origin xyz="-0.143415 0.122994 -0.0425" rpy="0 0 0"/>
+            <origin xyz="-0.4007 0.1312 -0.0425" rpy="0 0 0"/>
             <geometry>
                 <mesh filename="file://$(find ugv_description)/meshes/front_right_wheel.stl" scale="0.001 0.001 0.001"/>
@@ -76,5 +56,5 @@
         </visual>
         <collision>
-            <origin xyz="-0.143415 0.122994 -0.0425" rpy="0 0 0"/>
+            <origin xyz="-0.4007 0.1312 -0.0425" rpy="0 0 0"/>
             <geometry>
                 <mesh filename="file://$(find ugv_description)/meshes/front_right_wheel.stl" scale="0.001 0.001 0.001"/>
@@ -84,10 +64,10 @@
     <link name="rear_right_wheel">
         <inertial>
-            <origin xyz="1.2352069095333817e-07 -0.020000211992574915 2.9802314782667594e-10" rpy="0 0 0"/>
-            <mass value="1.578336149163512"/>
-            <inertia ixx="0.000842" iyy="0.001263" izz="0.000842" ixy="0.0" iyz="0.0" ixz="0.0"/>
+            <origin xyz="-3.1292413105177275e-10 -0.018799999999999956 2.9802320333782717e-10" rpy="0 0 0"/>
+            <mass value="1.4688367113110694"/>
+            <inertia ixx="0.000755" iyy="0.001163" izz="0.000755" ixy="0.0" iyz="0.0" ixz="0.0"/>
         </inertial>
         <visual>
-            <origin xyz="0.147785 0.122994 -0.0425" rpy="0 0 0"/>
+            <origin xyz="-0.1095 0.1312 -0.0425" rpy="0 0 0"/>
             <geometry>
                 <mesh filename="file://$(find ugv_description)/meshes/rear_right_wheel.stl" scale="0.001 0.001 0.001"/>
@@ -96,5 +76,5 @@
         </visual>
         <collision>
-            <origin xyz="0.147785 0.122994 -0.0425" rpy="0 0 0"/>
+            <origin xyz="-0.1095 0.1312 -0.0425" rpy="0 0 0"/>
             <geometry>
                 <mesh filename="file://$(find ugv_description)/meshes/rear_right_wheel.stl" scale="0.001 0.001 0.001"/>
@@ -102,38 +82,51 @@
         </collision>
     </link>
-    <link name="lidar_link">
+    <link name="rear_left_wheel">
         <inertial>
-            <origin xyz="-0.00011494677727549862 3.3107019681208537e-06 0.017944782112938054" rpy="0 0 0"/>
-            <mass value="0.7886321015037847"/>
-            <inertia ixx="0.000269" iyy="0.000272" izz="0.000333" ixy="0.0" iyz="0.0" ixz="-1e-06"/>
+            <origin xyz="-3.129242143184996e-10 0.01880000000000008 2.980232241545089e-10" rpy="0 0 0"/>
+            <mass value="1.4688367113110694"/>
+            <inertia ixx="0.000755" iyy="0.001163" izz="0.000755" ixy="0.0" iyz="0.0" ixz="0.0"/>
         </inertial>
         <visual>
-            <origin xyz="-0.186715 -6e-06 -0.091" rpy="0 0 0"/>
+            <origin xyz="-0.1095 -0.1148 -0.0425" rpy="0 0 0"/>
             <geometry>
-                <mesh filename="file://$(find ugv_description)/meshes/lidar_link.stl" scale="0.001 0.001 0.001"/>
+                <mesh filename="file://$(find ugv_description)/meshes/rear_left_wheel.stl" scale="0.001 0.001 0.001"/>
             </geometry>
             <material name="silver"/>
         </visual>
         <collision>
-            <origin xyz="-0.186715 -6e-06 -0.091" rpy="0 0 0"/>
+            <origin xyz="-0.1095 -0.1148 -0.0425" rpy="0 0 0"/>
             <geometry>
-                <mesh filename="file://$(find ugv_description)/meshes/lidar_link.stl" scale="0.001 0.001 0.001"/>
+                <mesh filename="file://$(find ugv_description)/meshes/rear_left_wheel.stl" scale="0.001 0.001 0.001"/>
             </geometry>
         </collision>
     </link>
-    <joint name="front_left_wheel_joint" type="continuous">
-        <origin xyz="0.143415 0.123006 0.0425" rpy="0 0 0"/>
+    <link name="front_left_wheel">
+        <inertial>
+            <origin xyz="-3.1292435309637767e-10 0.018800000000000303 2.980232241545089e-10" rpy="0 0 0"/>
+            <mass value="1.4688367113110694"/>
+            <inertia ixx="0.000755" iyy="0.001163" izz="0.000755" ixy="0.0" iyz="0.0" ixz="0.0"/>
+        </inertial>
+        <visual>
+            <origin xyz="-0.4007 -0.1148 -0.0425" rpy="0 0 0"/>
+            <geometry>
+                <mesh filename="file://$(find ugv_description)/meshes/front_left_wheel.stl" scale="0.001 0.001 0.001"/>
+            </geometry>
+            <material name="silver"/>
+        </visual>
+        <collision>
+            <origin xyz="-0.4007 -0.1148 -0.0425" rpy="0 0 0"/>
+            <geometry>
+                <mesh filename="file://$(find ugv_description)/meshes/front_left_wheel.stl" scale="0.001 0.001 0.001"/>
+            </geometry>
+        </collision>
+    </link>
+    <joint name="lidar_link_joint" type="fixed">
+        <origin xyz="0.43536 -6e-05 0.091" rpy="0 0 0"/>
         <parent link="base_link"/>
-        <child link="front_left_wheel"/>
-        <axis xyz="0.0 -1.0 0.0"/>
-    </joint>
-    <joint name="rear_left_wheel_joint" type="continuous">
-        <origin xyz="-0.147785 0.123006 0.0425" rpy="0 0 0"/>
-        <parent link="base_link"/>
-        <child link="rear_left_wheel"/>
-        <axis xyz="0.0 -1.0 0.0"/>
+        <child link="lidar_link"/>
     </joint>
     <joint name="front_right_wheel_joint" type="continuous">
-        <origin xyz="0.143415 -0.122994 0.0425" rpy="0 0 0"/>
+        <origin xyz="0.4007 -0.1312 0.0425" rpy="0 0 0"/>
         <parent link="base_link"/>
         <child link="front_right_wheel"/>
@@ -141,13 +134,20 @@
     </joint>
     <joint name="rear_right_wheel_joint" type="continuous">
-        <origin xyz="-0.147785 -0.122994 0.0425" rpy="0 0 0"/>
+        <origin xyz="0.1095 -0.1312 0.0425" rpy="0 0 0"/>
         <parent link="base_link"/>
         <child link="rear_right_wheel"/>
-        <axis xyz="-0.0 1.0 -0.0"/>
+        <axis xyz="-0.0 1.0 0.0"/>
     </joint>
-    <joint name="lidar_link_joint" type="fixed">
-        <origin xyz="0.186715 6e-06 0.091" rpy="0 0 0"/>
+    <joint name="rear_left_wheel_joint" type="continuous">
+        <origin xyz="0.1095 0.1148 0.0425" rpy="0 0 0"/>
         <parent link="base_link"/>
-        <child link="lidar_link"/>
+        <child link="rear_left_wheel"/>
+        <axis xyz="0.0 1.0 0.0"/>
+    </joint>
+    <joint name="front_left_wheel_joint" type="continuous">
+        <origin xyz="0.4007 0.1148 0.0425" rpy="0 0 0"/>
+        <parent link="base_link"/>
+        <child link="front_left_wheel"/>
+        <axis xyz="0.0 1.0 0.0"/>
     </joint>
     <link name="base_footprint"/>

Commit message: urdf lidar

File: ugv_description/urdf/ugv_core.xacro (robot description, xacro)
@@ -9,4 +9,7 @@
     <xacro:property name="wheel_thickness" value="0.0369" />
     <xacro:property name="wheel_mass" value="0.05" />
+    <xacro:property name="lidar_radius" value="0.04" />
+    <xacro:property name="lidar_thickness" value="0.0369" />
+    <xacro:property name="lidar_mass" value="0.05" />
     <xacro:property name="edge_to_motor_mount" value="0.04" />
     <xacro:property name="motor_mount_width" value="0.0417" />
@@ -39,4 +42,7 @@
         <color rgba="1 0.3 0.1 1" />
     </material>
+    <material name="yellow">
+        <color rgba="1 1 0 1" />
+    </material>
     <material name="black">
         <color rgba="0 0 0 1" />
@@ -58,5 +64,5 @@
         <xacro:inertial_box mass="${chassis_mass}" x="${chassis_length}" y="${chassis_width}"
             z="${chassis_height}">
-            <origin rpy="0 0 0" xyz="0 0 ${wheel_radius}"/>
+            <origin xyz="${chassis_length/2} 0 ${chassis_height/2}" rpy="0 0 0" />
         </xacro:inertial_box>
     </link>
@@ -99,29 +105,26 @@
         <axis xyz="0.0 1.0 0.0" />
     </joint>
-    <!--
     <link name="lidar_link">
-        <inertial>
-            <origin xyz="-0.0001155547326693318 3.2715051849067412e-06 0.01794478211293804" rpy="0 0 0"/>
-            <mass value="0.7886321015037847"/>
-            <inertia ixx="0.000269" iyy="0.000272" izz="0.000333" ixy="0.0" iyz="0.0" ixz="-1e-06"/>
-        </inertial>
         <visual>
-            <origin xyz="-0.43536 6e-05 -0.091" rpy="0 0 0"/>
+            <origin xyz="0 0 0" rpy="0 0 0"/>
             <geometry>
-                <mesh filename="file://$(find ugv_description)/meshes/lidar_link.stl" scale="0.001 0.001 0.001"/>
-            </geometry>
-            <material name="silver"/>
+                <cylinder radius="${lidar_radius}" length="${lidar_thickness}" />     </geometry>
+            <material name="yellow"/>
         </visual>
         <collision>
-            <origin xyz="-0.43536 6e-05 -0.091" rpy="0 0 0"/>
+            <origin xyz="0 0 0" rpy="0 0 0"/>
             <geometry>
-                <mesh filename="file://$(find ugv_description)/meshes/lidar_link.stl" scale="0.001 0.001 0.001"/>
+                <cylinder radius="${lidar_radius}" length="${lidar_thickness}" />
             </geometry>
         </collision>
+        <xacro:inertial_cylinder mass="${lidar_mass}" length="${lidar_thickness}"
+            radius="${lidar_radius}">
+            <origin xyz="0 0 0" rpy="0 0 0" />
+        </xacro:inertial_cylinder>
     </link>
     <joint name="lidar_link_joint" type="fixed">
         <parent link="base_link"/>
         <child link="lidar_link"/>
-        <origin xyz="0.43536 -6e-05 0.091" rpy="0 0 0"/>
-    </joint> -->
+        <origin xyz="${chassis_length/2} 0 ${wheel_radius}" rpy="0 0 0"/>
+    </joint>
 </robot>
