Commit message: lidar urdf

File: ugv_description/urdf/ugv_core.xacro (robot description, xacro)
@@ -2,11 +2,12 @@
 <robot name="ugv" xmlns:xacro="http://www.ros.org/wiki/xacro">
     <xacro:include filename="$(find ugv_description)/gazebo/common_inertias.xacro" />
+    <xacro:property name="wheel_radius" value="0.04" />
+    <xacro:property name="wheel_thickness" value="0.0369" />
+    <xacro:property name="wheel_mass" value="0.05" />
     <xacro:property name="chassis_length" value="0.34" />
     <xacro:property name="chassis_width" value="0.285" />
     <xacro:property name="chassis_height" value="0.02" />
     <xacro:property name="chassis_mass" value="1.0" />
-    <xacro:property name="wheel_radius" value="0.04" />
-    <xacro:property name="wheel_thickness" value="0.0369" />
-    <xacro:property name="wheel_mass" value="0.05" />
+    <xacro:property name="chassis_offset_z" value="${wheel_radius}" />
     <xacro:property name="lidar_radius" value="0.04" />
     <xacro:property name="lidar_thickness" value="0.0369" />
@@ -18,10 +19,10 @@
     <xacro:property name="wheel_offset_y" value="${chassis_width/2 + wheel_thickness/2 + 0.0029}"/>
     <xacro:property name="wheel_offset_z" value="0.01" />
-    <xacro:macro name="wheel" params="prefix mass radius thickness">
+    <xacro:macro name="wheel" params="prefix">
         <link name="${prefix}_wheel">
             <visual>
                 <origin rpy="${pi/2} 0 0" xyz="0 0 0"/>
                 <geometry>
-                    <cylinder radius="${radius}" length="${thickness}" />
+                    <cylinder radius="${wheel_radius}" length="${wheel_thickness}" />
                 </geometry>
                 <material name="orange" />
@@ -30,9 +31,9 @@
                 <origin rpy="${pi/2} 0 0" xyz="0 0 0"/>
                 <geometry>
-                    <cylinder radius="${radius}" length="${thickness}" />
+                    <cylinder radius="${wheel_radius}" length="${wheel_thickness}" />
                 </geometry>
             </collision>
-            <xacro:inertial_cylinder mass="${mass}" length="${thickness}"
-                radius="${radius}">
+            <xacro:inertial_cylinder mass="${wheel_mass}" length="${wheel_thickness}"
+                radius="${wheel_radius}">
                 <origin xyz="0 0 0" rpy="0 0 0" />
             </xacro:inertial_cylinder>
@@ -50,5 +51,5 @@
     <link name="base_link">
         <visual>
-            <origin rpy="0 0 0" xyz="0 0 ${wheel_radius}"/>
+            <origin rpy="0 0 0" xyz="0 0 ${chassis_offset_z}"/>
             <geometry>
                 <box size="${chassis_length} ${chassis_width} ${chassis_height}" />
@@ -57,5 +58,5 @@
         </visual>
         <collision>
-            <origin rpy="0 0 0" xyz="0 0 ${wheel_radius}"/>
+            <origin rpy="0 0 0" xyz="0 0 ${chassis_offset_z}"/>
             <geometry>
                 <box size="${chassis_length} ${chassis_width} ${chassis_height}" />
@@ -73,6 +74,5 @@
         <origin xyz="0 0 0" rpy="0 0 0" />
     </joint>
-    <xacro:wheel prefix="front_right" mass="${wheel_mass}" radius="${wheel_radius}"
-        thickness="${wheel_thickness}" />
+    <xacro:wheel prefix="front_right"  />
     <joint name="front_right_wheel_joint" type="continuous">
         <parent link="base_link" />
@@ -81,6 +81,5 @@
         <axis xyz="0.0 1.0 0.0" />
     </joint>
-    <xacro:wheel prefix="front_left" mass="${wheel_mass}" radius="${wheel_radius}"
-        thickness="${wheel_thickness}" />
+    <xacro:wheel prefix="front_left" />
     <joint name="front_left_wheel_joint" type="continuous">
         <parent link="base_link" />
@@ -89,6 +88,5 @@
         <axis xyz="0.0 1.0 0.0" />
     </joint>
-    <xacro:wheel prefix="rear_right" mass="${wheel_mass}" radius="${wheel_radius}"
-        thickness="${wheel_thickness}" />
+    <xacro:wheel prefix="rear_right"  />
     <joint name="rear_right_wheel_joint" type="continuous">
         <parent link="base_link" />
@@ -97,6 +95,5 @@
         <axis xyz="-0.0 1.0 0.0" />
     </joint>
-    <xacro:wheel prefix="rear_left" mass="${wheel_mass}" radius="${wheel_radius}"
-        thickness="${wheel_thickness}" />
+    <xacro:wheel prefix="rear_left" />
     <joint name="rear_left_wheel_joint" type="continuous">
         <parent link="base_link" />
@@ -126,5 +123,5 @@
         <parent link="base_link"/>
         <child link="lidar_link"/>
-        <origin xyz="${chassis_length/2} 0 ${wheel_radius}" rpy="0 0 0"/>
+        <origin xyz="${chassis_length/2-lidar_radius} 0 ${chassis_offset_z+chassis_height}" rpy="0 0 0"/>
     </joint>
 </robot>

Commit message: fixed inertia

File: ugv_description/urdf/ugv_core.xacro (robot description, xacro)
@@ -65,5 +65,5 @@
         <xacro:inertial_box mass="${chassis_mass}" x="${chassis_length}" y="${chassis_width}"
             z="${chassis_height}">
-            <origin xyz="${chassis_length/2} 0 ${chassis_height/2}" rpy="0 0 0" />
+            <origin rpy="0 0 0" xyz="0 0 ${chassis_offset_z}"/>
         </xacro:inertial_box>
     </link>

Commit message: Updated wheel_offset_x and wheel_offset_y

File: ugv_description/urdf/ugv_core.xacro (robot description, xacro)
@@ -13,9 +13,11 @@
     <xacro:property name="lidar_thickness" value="0.1" />
     <xacro:property name="lidar_mass" value="0.05" />
-    <xacro:property name="edge_to_motor_mount" value="0.04" />
+    <xacro:property name="edge_thickness" value="0.02" />
+    <xacro:property name="edge_to_motor_mount" value="0.016" />
     <xacro:property name="motor_mount_width" value="0.0417" />
-    <xacro:property name="motor_shaft_to_edge_x" value="${edge_to_motor_mount+motor_mount_width/2}" />
+    <xacro:property name="motor_shaft_to_edge_x" value="${edge_thickness+edge_to_motor_mount+motor_mount_width/2}" />
     <xacro:property name="wheel_offset_x" value="${chassis_length/2-motor_shaft_to_edge_x}" />
-    <xacro:property name="wheel_offset_y" value="${chassis_width/2 + wheel_thickness/2 + 0.0029}"/>
+    <xacro:property name="wheels_y_distance_edge_to_edge" value=".36"/>
+    <xacro:property name="wheel_offset_y" value="${wheels_y_distance_edge_to_edge/2 - wheel_thickness/2}"/>
     <xacro:property name="wheel_offset_z" value="0.01" />
     <xacro:macro name="wheel" params="prefix">

Commit message: .

File: ugv_description/urdf/ugv_core.xacro (robot description, xacro)
@@ -21,4 +21,13 @@
     <xacro:property name="wheel_offset_y" value="${wheels_y_distance_edge_to_edge/2 - wheel_thickness/2}"/>
     <xacro:property name="wheel_offset_z" value="0.01" />
+    <material name="orange">
+        <color rgba="1 0.3 0.1 1" />
+    </material>
+    <material name="yellow">
+        <color rgba="1 1 0 1" />
+    </material>
+    <material name="black">
+        <color rgba="0 0 0 1" />
+    </material>
     <xacro:macro name="wheel" params="prefix">
         <link name="${prefix}_wheel">
@@ -42,13 +51,4 @@
         </link>
     </xacro:macro>
-    <material name="orange">
-        <color rgba="1 0.3 0.1 1" />
-    </material>
-    <material name="yellow">
-        <color rgba="1 1 0 1" />
-    </material>
-    <material name="black">
-        <color rgba="0 0 0 1" />
-    </material>
     <link name="base_link">
         <visual>

Commit message: made base_footprint parent

File: ugv_description/urdf/ugv_core.xacro (robot description, xacro)
@@ -72,6 +72,6 @@
     <link name="base_footprint" />
     <joint name="base_footprint_joint" type="fixed">
-        <parent link="base_link" />
-        <child link="base_footprint" />
+        <parent link="base_footprint" />
+        <child link="base_link" />
         <origin xyz="0 0 0" rpy="0 0 0" />
     </joint>

Commit message: switched base_link nd base_footprint

File: ugv_description/urdf/ugv_core.xacro (robot description, xacro)
@@ -72,6 +72,6 @@
     <link name="base_footprint" />
     <joint name="base_footprint_joint" type="fixed">
-        <parent link="base_footprint" />
-        <child link="base_link" />
+        <parent link="base_link" />
+        <child link="base_footprint" />
         <origin xyz="0 0 0" rpy="0 0 0" />
     </joint>

Commit message: fixed lidar rotation!!

File: ugv_description/urdf/ugv_core.xacro (robot description, xacro)
@@ -125,5 +125,5 @@
         <parent link="base_link"/>
         <child link="lidar_link"/>
-        <origin xyz="${chassis_length/2-lidar_radius} 0 ${chassis_offset_z+lidar_thickness/2}" rpy="0 0 0"/>
+        <origin xyz="${chassis_length/2-lidar_radius} 0 ${chassis_offset_z+lidar_thickness/2}" rpy="0 0 ${pi}"/>
     </joint>
 </robot>

Commit message: updated wheel_radius in xacro

File: ugv_description/urdf/ugv_core.xacro (robot description, xacro)
@@ -2,5 +2,5 @@
 <robot name="ugv" xmlns:xacro="http://www.ros.org/wiki/xacro">
     <xacro:include filename="$(find ugv_description)/gazebo/common_inertias.xacro" />
-    <xacro:property name="wheel_radius" value="0.04" />
+    <xacro:property name="wheel_radius" value="0.0395" />
     <xacro:property name="wheel_thickness" value="0.0369" />
     <xacro:property name="wheel_mass" value="0.05" />
