Commit message: -common macro file

File: ugv_control/urdf/ugv.xacro (robot description, xacro)
@@ -2,5 +2,6 @@
 <robot name="ugv" xmlns:xacro="http://www.ros.org/wiki/xacro">
     <xacro:arg name="is_sim" default="true"/>
-    <xacro:include filename="$(find ugv_description)/urdf/ugv.xacro"/>
+    <xacro:include filename="$(find ugv_description)/urdf/ugv.macro.xacro"/>
+    <xacro:ugv is_sim="$is_sim"/>
     <xacro:if value="$(arg is_sim)">
         <xacro:include filename="$(find ugv_control)/urdf/gazebo_control.xacro"/>

File: ugv_description/gazebo/gazebo.xacro (robot description, xacro)
@@ -2,4 +2,5 @@
 <robot name="ugv" xmlns:xacro="http://www.ros.org/wiki/xacro">
     <xacro:property name="body_color" value="Gazebo/Silver"/>
+    <xacro:property name="wheels_color" value="Gazebo/Yellow"/>
     <gazebo reference="base_link">
         <material>${body_color}</material>
@@ -33,9 +34,3 @@
         <self_collide>true</self_collide>
     </gazebo>
-    <gazebo reference="lidar_link">
-        <material>${body_color}</material>
-        <mu1>0.2</mu1>
-        <mu2>0.2</mu2>
-        <self_collide>true</self_collide>
-    </gazebo>
 </robot>

File: ugv_description/gazebo/lidar.xacro (robot description, xacro)
@@ -3,4 +3,7 @@
     <gazebo reference="lidar_link">
         <material>Gazebo/Black</material>
+        <mu1>0.2</mu1>
+        <mu2>0.2</mu2>
+        <self_collide>true</self_collide>
         <sensor name="laser" type="ray">
             <pose>0 0 0 0 0 0</pose>

File: ugv_description/urdf/ugv.xacro (robot description, xacro)
@@ -2,9 +2,5 @@
 <robot name="ugv" xmlns:xacro="http://www.ros.org/wiki/xacro">
     <xacro:arg name="is_sim" default="true"/>
-    <xacro:include filename="ugv_core.xacro"/>
-    <xacro:if value="$(arg is_sim)">
-        <xacro:include filename="$(find ugv_description)/gazebo/gazebo.xacro"/>
-        <xacro:include filename="$(find ugv_description)/gazebo/lidar.xacro"/>
-        <!--        <xacro:include filename="gazebo/imu.xacro"/>-->
-    </xacro:if>
+    <xacro:include filename="$(find ugv_description)/urdf/ugv.macro.xacro"/>
+    <xacro:ugv is_sim="$is_sim"/>
 </robot>
