Commit message: disabled front_left_wheel_joint and front_right_wheel_joint

File: ugv_control/urdf/joints.macro.xacro (robot description, xacro)
@@ -2,5 +2,5 @@
 <robot xmlns:xacro="http://www.ros.org/wiki/xacro">
     <xacro:macro name="joints">
-        <joint name="front_left_wheel_joint">
+        <!-- <joint name="front_left_wheel_joint">
             <command_interface name="velocity"/>
             <state_interface name="position"/>
@@ -9,5 +9,5 @@
             <command_interface name="velocity"/>
             <state_interface name="position"/>
-        </joint>
+        </joint> -->
         <joint name="rear_left_wheel_joint">
             <command_interface name="velocity"/>

Commit message: fixed urdf + inertia

File: ugv_control/urdf/joints.macro.xacro (robot description, xacro)
@@ -2,5 +2,5 @@
 <robot xmlns:xacro="http://www.ros.org/wiki/xacro">
     <xacro:macro name="joints">
-        <!-- <joint name="front_left_wheel_joint">
+        <joint name="front_left_wheel_joint">
             <command_interface name="velocity"/>
             <state_interface name="position"/>
@@ -9,5 +9,5 @@
             <command_interface name="velocity"/>
             <state_interface name="position"/>
-        </joint> -->
+        </joint>
         <joint name="rear_left_wheel_joint">
             <command_interface name="velocity"/>

File: ugv_description/gazebo/common_inertias.xacro (robot description, xacro)
@@ -1,61 +1,32 @@
 <?xml version="1.0"?>
 <robot xmlns:xacro="http://www.ros.org/wiki/xacro">
-    <!-- see https://secure.wikimedia.org/wikipedia/en/wiki/List_of_moment_of_inertia_tensors -->
-    <xacro:macro name="sphere_inertial" params="radius mass *origin">
+    <!-- Specify some standard inertial calculations
+    https://en.wikipedia.org/wiki/List_of_moments_of_inertia -->
+    <!-- These make use of xacro's mathematical functionality -->
+    <xacro:macro name="inertial_sphere" params="mass radius *origin">
         <inertial>
-            <mass value="${mass}"/>
-            <xacro:insert_block name="origin"/>
-            <inertia ixx="${2.0/5 * mass * radius * radius}" ixy="0.0" ixz="0.0"
-                     iyy="${2.0/5 * mass * radius * radius}" iyz="0.0"
-                     izz="${2.0/5 * mass * radius * radius}"/>
+            <xacro:insert_block name="origin" />
+            <mass value="${mass}" />
+            <inertia ixx="${(2/5) * mass * (radius*radius)}" ixy="0.0" ixz="0.0"
+                iyy="${(2/5) * mass * (radius*radius)}" iyz="0.0"
+                izz="${(2/5) * mass * (radius*radius)}" />
         </inertial>
     </xacro:macro>
-    <xacro:macro name="cylinder_inertial" params="radius length mass rotation">
+    <xacro:macro name="inertial_box" params="mass x y z *origin">
         <inertial>
-            <origin xyz="0 0 0" rpy="${rotation} 0 0"/>
-            <mass value="${mass}"/>
-            <inertia ixx="${1.0/12 * mass * (3 * radius * radius + length * length)}" ixy="0.0" ixz="0.0"
-                     iyy="${1.0/12 * mass * (3 * radius * radius + length * length)}" iyz="0.0"
-                     izz="${1.0/2 * mass * radius * radius}"/>
+            <xacro:insert_block name="origin" />
+            <mass value="${mass}" />
+            <inertia ixx="${(1/12) * mass * (y*y+z*z)}" ixy="0.0" ixz="0.0"
+                iyy="${(1/12) * mass * (x*x+z*z)}" iyz="0.0"
+                izz="${(1/12) * mass * (x*x+y*y)}" />
         </inertial>
     </xacro:macro>
-    <xacro:macro name="box_inertial" params="x y z mass ">
+    <xacro:macro name="inertial_cylinder" params="mass length radius *origin">
         <inertial>
-            <mass value="${mass}"/>
-            <inertia ixx="${1.0/12 * mass * (y*y + z*z)}" ixy="0.0" ixz="0.0"
-                     iyy="${1.0/12 * mass * (x*x + z*z)}" iyz="0.0"
-                     izz="${1.0/12 * mass * (x*x + y*y)}"/>
-        </inertial>
-    </xacro:macro>
-    <xacro:macro name="spherical_cap_inertial" params="r h mass *origin">
-        <inertial>
-            <mass value="${mass}"/>
-            <xacro:insert_block name="origin"/>
-            <inertia
-                    ixx="${(-3*h*h*h/20+3*h*h*r/4-4*h*r*r/3+r*r*r)*3*mass/(3*r-h)+(3/4*(h-2*r)*(h-2*r)/(3*r-h))*(3/4*(h-2*r)*(h-2*r)/(3*r-h))}"
-                    ixy="0.0" ixz="0.0"
-                    iyy="${(-3*h*h*h/20+3*h*h*r/4-4*h*r*r/3+r*r*r)*3*mass/(3*r-h)+(3/4*(h-2*r)*(h-2*r)/(3*r-h))*(3/4*(h-2*r)*(h-2*r)/(3*r-h))}"
-                    iyz="0.0"
-                    izz="${mass*h/(10*(3*r-h))*(3*h*h-15*h*r+20*r*r)}"/>
-            <origin></origin>
-        </inertial>
-    </xacro:macro>
-    <xacro:macro name="hollow_spherical_cap_inertial" params="r h t mass *origin">
-        <inertial>
-            <mass value="${mass}"/>
-            <xacro:insert_block name="origin"/>
-            <inertia
-                    ixx="${mass/20*(20*h*h*h*r-10*h*h*h*t-60*h*h*r*r+30*h*h*r*t+120*h*r*r*r-120*h*r*r*t+60*h*r*t*t-15*h*t*t*t-60*r*r*r*t+100*r*r*t*t-65*r*t*t*t+16*t*t*t*t)/(2*t*t*-3*r*t-3*h*t+6*h*r)+(3/4*(t-2*r)*(2*r*r-4*r*r+2*r*t-t*t)/(6*r*r-3*r*t-3*r*t+2*t*t))*(3/4*(t-2*r)*(2*r*r-4*r*r+2*r*t-t*t)/(6*r*r-3*r*t-3*r*t+2*t*t))}"
-                    ixy="0.0" ixz="0.0"
-                    iyy="${mass/20*(20*h*h*h*r-10*h*h*h*t-60*h*h*r*r+30*h*h*r*t+120*h*r*r*r-120*h*r*r*t+60*h*r*t*t-15*h*t*t*t-60*r*r*r*t+100*r*r*t*t-65*r*t*t*t+16*t*t*t*t)/(2*t*t*-3*r*t-3*h*t+6*h*r)+(3/4*(t-2*r)*(2*r*r-4*r*r+2*r*t-t*t)/(6*r*r-3*r*t-3*r*t+2*t*t))*(3/4*(t-2*r)*(2*r*r-4*r*r+2*r*t-t*t)/(6*r*r-3*r*t-3*r*t+2*t*t))}"
-                    iyz="0.0"
-                    izz="${mass/(10*(2*t*t-3*r*t-3*h*t+6*h*r))*(-20*h*h*h*r+10*h*h*h*t+60*h*h*r*r-30*h*h*r*t-60*h*r*r*t+60*h*r*t*t-15*h*t*t*t+20*r*r*t*t-25*r*t*t*t+8*t*t*t*t)}"/>
-        </inertial>
-    </xacro:macro>
-    <xacro:macro name="default_inertial">
-        <inertial>
-            <mass value="0.01"/>
-            <origin xyz="0 0 0"/>
-            <inertia ixx="0.001" ixy="0.0" ixz="0.0" iyy="0.001" iyz="0.0" izz="0.001"/>
+            <xacro:insert_block name="origin" />
+            <mass value="${mass}" />
+            <inertia ixx="${(1/12) * mass * (3*radius*radius + length*length)}" ixy="0.0" ixz="0.0"
+                iyy="${(1/12) * mass * (3*radius*radius + length*length)}" iyz="0.0"
+                izz="${(1/2) * mass * (radius*radius)}" />
         </inertial>
     </xacro:macro>

File: ugv_description/urdf/ugv_core.xacro (robot description, xacro)
@@ -1,25 +1,103 @@
-<?xml version="1.0" ?>
+<?xml version="1.0"?>
 <robot name="ugv" xmlns:xacro="http://www.ros.org/wiki/xacro">
-    <xacro:include filename="$(find ugv_description)/urdf/materials.xacro"/>
+    <xacro:include filename="$(find ugv_description)/gazebo/common_inertias.xacro" />
+    <xacro:property name="chassis_length" value="0.34" />
+    <xacro:property name="chassis_width" value="0.285" />
+    <xacro:property name="chassis_height" value="0.02" />
+    <xacro:property name="chassis_mass" value="1.0" />
+    <xacro:property name="wheel_radius" value="0.04" />
+    <xacro:property name="wheel_thickness" value="0.0369" />
+    <xacro:property name="wheel_mass" value="0.05" />
+    <xacro:property name="edge_to_motor_mount" value="0.04" />
+    <xacro:property name="motor_mount_width" value="0.0417" />
+    <xacro:property name="motor_shaft_to_edge_x" value="${edge_to_motor_mount+motor_mount_width/2}" />
+    <xacro:property name="wheel_offset_x" value="${chassis_length/2-motor_shaft_to_edge_x}" />
+    <xacro:property name="wheel_offset_y" value="${chassis_width/2 + wheel_thickness/2 + 0.0029}"/>
+    <xacro:property name="wheel_offset_z" value="0.01" />
+    <xacro:macro name="wheel" params="prefix mass radius thickness">
+        <link name="${prefix}_wheel">
+            <visual>
+                <origin rpy="${pi/2} 0 0" xyz="0 0 0"/>
+                <geometry>
+                    <cylinder radius="${radius}" length="${thickness}" />
+                </geometry>
+                <material name="orange" />
+            </visual>
+            <collision>
+                <origin rpy="${pi/2} 0 0" xyz="0 0 0"/>
+                <geometry>
+                    <cylinder radius="${radius}" length="${thickness}" />
+                </geometry>
+            </collision>
+            <xacro:inertial_cylinder mass="${mass}" length="${thickness}"
+                radius="${radius}">
+                <origin xyz="0 0 0" rpy="0 0 0" />
+            </xacro:inertial_cylinder>
+        </link>
+    </xacro:macro>
+    <material name="orange">
+        <color rgba="1 0.3 0.1 1" />
+    </material>
+    <material name="black">
+        <color rgba="0 0 0 1" />
+    </material>
     <link name="base_link">
-        <inertial>
-            <origin xyz="0.25539221363619424 -0.008191452128420306 0.07740258559841702" rpy="0 0 0"/>
-            <mass value="1.8582255296411472"/>
-            <inertia ixx="0.018307" iyy="0.036178" izz="0.054" ixy="-3e-06" iyz="-0.0" ixz="-5e-06"/>
-        </inertial>
         <visual>
-            <origin xyz="0 0 0" rpy="0 0 0"/>
+            <origin rpy="0 0 0" xyz="0 0 ${wheel_radius}"/>
             <geometry>
-                <mesh filename="file://$(find ugv_description)/meshes/base_link.stl" scale="0.001 0.001 0.001"/>
+                <box size="${chassis_length} ${chassis_width} ${chassis_height}" />
             </geometry>
-            <material name="silver"/>
+            <material name="black" />
         </visual>
         <collision>
-            <origin xyz="0 0 0" rpy="0 0 0"/>
+            <origin rpy="0 0 0" xyz="0 0 ${wheel_radius}"/>
             <geometry>
-                <mesh filename="file://$(find ugv_description)/meshes/base_link.stl" scale="0.001 0.001 0.001"/>
+                <box size="${chassis_length} ${chassis_width} ${chassis_height}" />
             </geometry>
         </collision>
+        <xacro:inertial_box mass="${chassis_mass}" x="${chassis_length}" y="${chassis_width}"
+            z="${chassis_height}">
+            <origin rpy="0 0 0" xyz="0 0 ${wheel_radius}"/>
+        </xacro:inertial_box>
     </link>
+    <link name="base_footprint" />
+    <joint name="base_footprint_joint" type="fixed">
+        <parent link="base_link" />
+        <child link="base_footprint" />
+        <origin xyz="0 0 0" rpy="0 0 0" />
+    </joint>
+    <xacro:wheel prefix="front_right" mass="${wheel_mass}" radius="${wheel_radius}"
+        thickness="${wheel_thickness}" />
+    <joint name="front_right_wheel_joint" type="continuous">
+        <parent link="base_link" />
+        <child link="front_right_wheel" />
+        <origin xyz="${wheel_offset_x} ${-wheel_offset_y} ${wheel_radius}" />
+        <axis xyz="0.0 1.0 0.0" />
+    </joint>
+    <xacro:wheel prefix="front_left" mass="${wheel_mass}" radius="${wheel_radius}"
+        thickness="${wheel_thickness}" />
+    <joint name="front_left_wheel_joint" type="continuous">
+        <parent link="base_link" />
+        <child link="front_left_wheel" />
+        <origin xyz="${wheel_offset_x} ${wheel_offset_y} ${wheel_radius}" />
+        <axis xyz="0.0 1.0 0.0" />
+    </joint>
+    <xacro:wheel prefix="rear_right" mass="${wheel_mass}" radius="${wheel_radius}"
+        thickness="${wheel_thickness}" />
+    <joint name="rear_right_wheel_joint" type="continuous">
+        <parent link="base_link" />
+        <child link="rear_right_wheel" />
+        <origin xyz="${-wheel_offset_x} ${-wheel_offset_y} ${wheel_radius}" />
+        <axis xyz="-0.0 1.0 0.0" />
+    </joint>
+    <xacro:wheel prefix="rear_left" mass="${wheel_mass}" radius="${wheel_radius}"
+        thickness="${wheel_thickness}" />
+    <joint name="rear_left_wheel_joint" type="continuous">
+        <parent link="base_link" />
+        <child link="rear_left_wheel" />
+        <origin xyz="${-wheel_offset_x} ${wheel_offset_y} ${wheel_radius}" />
+        <axis xyz="0.0 1.0 0.0" />
+    </joint>
+    <!--
     <link name="lidar_link">
         <inertial>
@@ -42,118 +120,8 @@
         </collision>
     </link>
-    <link name="front_right_wheel">
-        <inertial>
-            <origin xyz="-3.129242420740752e-10 -0.018799999999999678 2.9802320333782717e-10" rpy="0 0 0"/>
-            <mass value="1.4688367113110694"/>
-            <inertia ixx="0.000755" iyy="0.001163" izz="0.000755" ixy="0.0" iyz="0.0" ixz="-0.0"/>
-        </inertial>
-        <visual>
-            <origin xyz="-0.4007 0.1312 -0.0425" rpy="0 0 0"/>
-            <geometry>
-                <mesh filename="file://$(find ugv_description)/meshes/front_right_wheel.stl" scale="0.001 0.001 0.001"/>
-            </geometry>
-            <material name="silver"/>
-        </visual>
-        <collision>
-            <origin xyz="-0.4007 0.1312 -0.0425" rpy="0 0 0"/>
-            <geometry>
-                <mesh filename="file://$(find ugv_description)/meshes/front_right_wheel.stl" scale="0.001 0.001 0.001"/>
-            </geometry>
-        </collision>
-    </link>
-    <link name="rear_right_wheel">
-        <inertial>
-            <origin xyz="-3.1292413105177275e-10 -0.018799999999999956 2.9802320333782717e-10" rpy="0 0 0"/>
-            <mass value="1.4688367113110694"/>
-            <inertia ixx="0.000755" iyy="0.001163" izz="0.000755" ixy="0.0" iyz="0.0" ixz="0.0"/>
-        </inertial>
-        <visual>
-            <origin xyz="-0.1095 0.1312 -0.0425" rpy="0 0 0"/>
-            <geometry>
-                <mesh filename="file://$(find ugv_description)/meshes/rear_right_wheel.stl" scale="0.001 0.001 0.001"/>
-            </geometry>
-            <material name="silver"/>
-        </visual>
-        <collision>
-            <origin xyz="-0.1095 0.1312 -0.0425" rpy="0 0 0"/>
-            <geometry>
-                <mesh filename="file://$(find ugv_description)/meshes/rear_right_wheel.stl" scale="0.001 0.001 0.001"/>
-            </geometry>
-        </collision>
-    </link>
-    <link name="rear_left_wheel">
-        <inertial>
-            <origin xyz="-3.129242143184996e-10 0.01880000000000008 2.980232241545089e-10" rpy="0 0 0"/>
-            <mass value="1.4688367113110694"/>
-            <inertia ixx="0.000755" iyy="0.001163" izz="0.000755" ixy="0.0" iyz="0.0" ixz="0.0"/>
-        </inertial>
-        <visual>
-            <origin xyz="-0.1095 -0.1148 -0.0425" rpy="0 0 0"/>
-            <geometry>
-                <mesh filename="file://$(find ugv_description)/meshes/rear_left_wheel.stl" scale="0.001 0.001 0.001"/>
-            </geometry>
-            <material name="silver"/>
-        </visual>
-        <collision>
-            <origin xyz="-0.1095 -0.1148 -0.0425" rpy="0 0 0"/>
-            <geometry>
-                <mesh filename="file://$(find ugv_description)/meshes/rear_left_wheel.stl" scale="0.001 0.001 0.001"/>
-            </geometry>
-        </collision>
-    </link>
-    <link name="front_left_wheel">
-        <inertial>
-            <origin xyz="-3.1292435309637767e-10 0.018800000000000303 2.980232241545089e-10" rpy="0 0 0"/>
-            <mass value="1.4688367113110694"/>
-            <inertia ixx="0.000755" iyy="0.001163" izz="0.000755" ixy="0.0" iyz="0.0" ixz="0.0"/>
-        </inertial>
-        <visual>
-            <origin xyz="-0.4007 -0.1148 -0.0425" rpy="0 0 0"/>
-            <geometry>
-                <mesh filename="file://$(find ugv_description)/meshes/front_left_wheel.stl" scale="0.001 0.001 0.001"/>
-            </geometry>
-            <material name="silver"/>
-        </visual>
-        <collision>
-            <origin xyz="-0.4007 -0.1148 -0.0425" rpy="0 0 0"/>
-            <geometry>
-                <mesh filename="file://$(find ugv_description)/meshes/front_left_wheel.stl" scale="0.001 0.001 0.001"/>
-            </geometry>
-        </collision>
-    </link>
     <joint name="lidar_link_joint" type="fixed">
-        <origin xyz="0.43536 -6e-05 0.091" rpy="0 0 0"/>
         <parent link="base_link"/>
         <child link="lidar_link"/>
-    </joint>
-    <joint name="front_right_wheel_joint" type="continuous">
-        <origin xyz="0.4007 -0.1312 0.0425" rpy="0 0 0"/>
-        <parent link="base_link"/>
-        <child link="front_right_wheel"/>
-        <axis xyz="-0.0 1.0 -0.0"/>
-    </joint>
-    <joint name="rear_right_wheel_joint" type="continuous">
-        <origin xyz="0.1095 -0.1312 0.0425" rpy="0 0 0"/>
-        <parent link="base_link"/>
-        <child link="rear_right_wheel"/>
-        <axis xyz="-0.0 1.0 0.0"/>
-    </joint>
-    <joint name="rear_left_wheel_joint" type="continuous">
-        <origin xyz="0.1095 0.1148 0.0425" rpy="0 0 0"/>
-        <parent link="base_link"/>
-        <child link="rear_left_wheel"/>
-        <axis xyz="0.0 1.0 0.0"/>
-    </joint>
-    <joint name="front_left_wheel_joint" type="continuous">
-        <origin xyz="0.4007 0.1148 0.0425" rpy="0 0 0"/>
-        <parent link="base_link"/>
-        <child link="front_left_wheel"/>
-        <axis xyz="0.0 1.0 0.0"/>
-    </joint>
-    <link name="base_footprint"/>
-    <joint name="base_footprint_joint" type="fixed">
-        <parent link="base_link"/>
-        <child link="base_footprint"/>
-        <origin xyz="0 0 0" rpy="0 0 0"/>
-    </joint>
+        <origin xyz="0.43536 -6e-05 0.091" rpy="0 0 0"/>
+    </joint> -->
 </robot>
