Commit message: lidar

File: ugv_description/gazebo/lidar.xacro (robot description, xacro)
@@ -10,4 +10,5 @@
             <visualize>true</visualize>
             <update_rate>10</update_rate>
+            <always_on>1</always_on>
             <ray>
                 <scan>

File: ugv_description/urdf/ugv_core.xacro (robot description, xacro)
@@ -10,6 +10,6 @@
     <xacro:property name="chassis_mass" value="1.0" />
     <xacro:property name="chassis_offset_z" value="${wheel_radius}" />
-    <xacro:property name="lidar_radius" value="0.04" />
-    <xacro:property name="lidar_thickness" value="0.0369" />
+    <xacro:property name="lidar_radius" value="0.02" />
+    <xacro:property name="lidar_thickness" value="0.1" />
     <xacro:property name="lidar_mass" value="0.05" />
     <xacro:property name="edge_to_motor_mount" value="0.04" />
@@ -123,5 +123,5 @@
         <parent link="base_link"/>
         <child link="lidar_link"/>
-        <origin xyz="${chassis_length/2-lidar_radius} 0 ${chassis_offset_z+chassis_height}" rpy="0 0 0"/>
+        <origin xyz="${chassis_length/2-lidar_radius} 0 ${chassis_offset_z+lidar_thickness/2}" rpy="0 0 0"/>
     </joint>
 </robot>
