Commit message: -removed _1 postfix from wheels' names -using bool in launch files

File: ugv_description/gazebo/gazebo.xacro (robot description, xacro)
@@ -9,5 +9,5 @@
         <gravity>true</gravity>
     </gazebo>
-    <gazebo reference="front_left_wheel_1">
+    <gazebo reference="front_left_wheel">
         <material>${body_color}</material>
         <mu1>0.2</mu1>
@@ -15,5 +15,5 @@
         <self_collide>true</self_collide>
     </gazebo>
-    <gazebo reference="rear_left_wheel_1">
+    <gazebo reference="rear_left_wheel">
         <material>${body_color}</material>
         <mu1>0.2</mu1>
@@ -21,5 +21,5 @@
         <self_collide>true</self_collide>
     </gazebo>
-    <gazebo reference="rear_right_wheel_1">
+    <gazebo reference="rear_right_wheel">
         <material>${body_color}</material>
         <mu1>0.2</mu1>
@@ -27,5 +27,5 @@
         <self_collide>true</self_collide>
     </gazebo>
-    <gazebo reference="front_right_wheel_1">
+    <gazebo reference="front_right_wheel">
         <material>${body_color}</material>
         <mu1>0.2</mu1>
@@ -33,5 +33,5 @@
         <self_collide>true</self_collide>
     </gazebo>
-    <gazebo reference="lidar_link_1">
+    <gazebo reference="lidar_link">
         <material>${body_color}</material>
         <mu1>0.2</mu1>

File: ugv_description/urdf/ugv_core.xacro (robot description, xacro)
@@ -22,5 +22,5 @@
         </collision>
     </link>
-    <link name="front_left_wheel_1">
+    <link name="front_left_wheel">
         <inertial>
             <origin xyz="0.0 0.018500000000000072 -6.938893903907228e-18" rpy="0 0 0"/>
@@ -31,5 +31,5 @@
             <origin xyz="-0.09841 -0.125 -0.02" rpy="0 0 0"/>
             <geometry>
-                <mesh filename="file://$(find ugv_description)/meshes/front_left_wheel_1.stl"
+                <mesh filename="file://$(find ugv_description)/meshes/front_left_wheel.stl"
                       scale="0.001 0.001 0.001"/>
             </geometry>
@@ -39,10 +39,10 @@
             <origin xyz="-0.09841 -0.125 -0.02" rpy="0 0 0"/>
             <geometry>
-                <mesh filename="file://$(find ugv_description)/meshes/front_left_wheel_1.stl"
+                <mesh filename="file://$(find ugv_description)/meshes/front_left_wheel.stl"
                       scale="0.001 0.001 0.001"/>
             </geometry>
         </collision>
     </link>
-    <link name="rear_left_wheel_1">
+    <link name="rear_left_wheel">
         <inertial>
             <origin xyz="-1.3877787807814457e-17 0.018500000000000072 -6.938893903907228e-18" rpy="0 0 0"/>
@@ -53,5 +53,5 @@
             <origin xyz="0.09841 -0.125 -0.02" rpy="0 0 0"/>
             <geometry>
-                <mesh filename="file://$(find ugv_description)/meshes/rear_left_wheel_1.stl" scale="0.001 0.001 0.001"/>
+                <mesh filename="file://$(find ugv_description)/meshes/rear_left_wheel.stl" scale="0.001 0.001 0.001"/>
             </geometry>
             <material name="silver"/>
@@ -60,9 +60,9 @@
             <origin xyz="0.09841 -0.125 -0.02" rpy="0 0 0"/>
             <geometry>
-                <mesh filename="file://$(find ugv_description)/meshes/rear_left_wheel_1.stl" scale="0.001 0.001 0.001"/>
+                <mesh filename="file://$(find ugv_description)/meshes/rear_left_wheel.stl" scale="0.001 0.001 0.001"/>
             </geometry>
         </collision>
     </link>
-    <link name="rear_right_wheel_1">
+    <link name="rear_right_wheel">
         <inertial>
             <origin xyz="-1.3877787807814457e-17 -0.01849999999999999 -6.938893903907228e-18" rpy="0 0 0"/>
@@ -73,5 +73,5 @@
             <origin xyz="0.09841 0.125 -0.02" rpy="0 0 0"/>
             <geometry>
-                <mesh filename="file://$(find ugv_description)/meshes/rear_right_wheel_1.stl"
+                <mesh filename="file://$(find ugv_description)/meshes/rear_right_wheel.stl"
                       scale="0.001 0.001 0.001"/>
             </geometry>
@@ -81,10 +81,10 @@
             <origin xyz="0.09841 0.125 -0.02" rpy="0 0 0"/>
             <geometry>
-                <mesh filename="file://$(find ugv_description)/meshes/rear_right_wheel_1.stl"
+                <mesh filename="file://$(find ugv_description)/meshes/rear_right_wheel.stl"
                       scale="0.001 0.001 0.001"/>
             </geometry>
         </collision>
     </link>
-    <link name="front_right_wheel_1">
+    <link name="front_right_wheel">
         <inertial>
             <origin xyz="-1.1102230246251565e-15 -0.018500000000000072 -6.938893903907228e-18" rpy="0 0 0"/>
@@ -95,5 +95,5 @@
             <origin xyz="-0.09841 0.125 -0.02" rpy="0 0 0"/>
             <geometry>
-                <mesh filename="file://$(find ugv_description)/meshes/front_right_wheel_1.stl"
+                <mesh filename="file://$(find ugv_description)/meshes/front_right_wheel.stl"
                       scale="0.001 0.001 0.001"/>
             </geometry>
@@ -103,10 +103,10 @@
             <origin xyz="-0.09841 0.125 -0.02" rpy="0 0 0"/>
             <geometry>
-                <mesh filename="file://$(find ugv_description)/meshes/front_right_wheel_1.stl"
+                <mesh filename="file://$(find ugv_description)/meshes/front_right_wheel.stl"
                       scale="0.001 0.001 0.001"/>
             </geometry>
         </collision>
     </link>
-    <link name="lidar_link_1">
+    <link name="lidar_link">
         <inertial>
             <origin xyz="0.0 7.237528875152536e-18 0.009999999999999995" rpy="0 0 0"/>
@@ -117,5 +117,5 @@
             <origin xyz="-0.12 -0.0 -0.11" rpy="0 0 0"/>
             <geometry>
-                <mesh filename="file://$(find ugv_description)/meshes/lidar_link_1.stl" scale="0.001 0.001 0.001"/>
+                <mesh filename="file://$(find ugv_description)/meshes/lidar_link.stl" scale="0.001 0.001 0.001"/>
             </geometry>
             <material name="silver"/>
@@ -124,5 +124,5 @@
             <origin xyz="-0.12 -0.0 -0.11" rpy="0 0 0"/>
             <geometry>
-                <mesh filename="file://$(find ugv_description)/meshes/lidar_link_1.stl" scale="0.001 0.001 0.001"/>
+                <mesh filename="file://$(find ugv_description)/meshes/lidar_link.stl" scale="0.001 0.001 0.001"/>
             </geometry>
         </collision>
@@ -131,5 +131,5 @@
         <origin xyz="0.09841 0.125 0.02" rpy="0 0 0"/>
         <parent link="base_link"/>
-        <child link="front_left_wheel_1"/>
+        <child link="front_left_wheel"/>
         <axis xyz="0.0 -1.0 0.0"/>
     </joint>
@@ -137,5 +137,5 @@
         <origin xyz="-0.09841 0.125 0.02" rpy="0 0 0"/>
         <parent link="base_link"/>
-        <child link="rear_left_wheel_1"/>
+        <child link="rear_left_wheel"/>
         <axis xyz="0.0 1.0 0.0"/>
     </joint>
@@ -143,5 +143,5 @@
         <origin xyz="-0.09841 -0.125 0.02" rpy="0 0 0"/>
         <parent link="base_link"/>
-        <child link="rear_right_wheel_1"/>
+        <child link="rear_right_wheel"/>
         <axis xyz="0.0 1.0 0.0"/>
     </joint>
@@ -149,5 +149,5 @@
         <origin xyz="0.09841 -0.125 0.02" rpy="0 0 0"/>
         <parent link="base_link"/>
-        <child link="front_right_wheel_1"/>
+        <child link="front_right_wheel"/>
         <axis xyz="0.0 -1.0 0.0"/>
     </joint>
@@ -155,5 +155,5 @@
         <origin xyz="0.12 0.0 0.11" rpy="0 0 0"/>
         <parent link="base_link"/>
-        <child link="lidar_link_1"/>
+        <child link="lidar_link"/>
     </joint>
     <link name="base_footprint"/>

Commit message: -gazebo wheel colours

File: ugv_description/gazebo/gazebo.xacro (robot description, xacro)
@@ -11,5 +11,5 @@
     </gazebo>
     <gazebo reference="front_left_wheel">
-        <material>${body_color}</material>
+        <material>${wheels_color}</material>
         <mu1>0.2</mu1>
         <mu2>0.2</mu2>
@@ -17,5 +17,5 @@
     </gazebo>
     <gazebo reference="rear_left_wheel">
-        <material>${body_color}</material>
+        <material>${wheels_color}</material>
         <mu1>0.2</mu1>
         <mu2>0.2</mu2>
@@ -23,5 +23,5 @@
     </gazebo>
     <gazebo reference="rear_right_wheel">
-        <material>${body_color}</material>
+        <material>${wheels_color}</material>
         <mu1>0.2</mu1>
         <mu2>0.2</mu2>
@@ -29,5 +29,5 @@
     </gazebo>
     <gazebo reference="front_right_wheel">
-        <material>${body_color}</material>
+        <material>${wheels_color}</material>
         <mu1>0.2</mu1>
         <mu2>0.2</mu2>

Commit message: migrate to gazebo harmonic

File: ugv_description/gazebo/gazebo.xacro (robot description, xacro)
@@ -1,28 +1,47 @@
 <?xml version="1.0" ?>
-<robot name="ugv" xmlns:xacro="http://www.ros.org/wiki/xacro">
-    <xacro:property name="body_color" value="Gazebo/Silver"/>
-    <xacro:property name="wheels_color" value="Gazebo/Yellow"/>
-    <gazebo reference="base_link">
-        <material>${body_color}</material>
-    </gazebo>
-    <gazebo reference="front_left_wheel">
-        <material>${wheels_color}</material>
-        <mu1>0.001</mu1>
-        <mu2>0.001</mu2>
-    </gazebo>
-    <gazebo reference="rear_left_wheel">
-        <material>${wheels_color}</material>
-        <mu1>0.001</mu1>
-        <mu2>0.001</mu2>
-    </gazebo>
-    <gazebo reference="rear_right_wheel">
-        <material>${wheels_color}</material>
-        <mu1>0.001</mu1>
-        <mu2>0.001</mu2>
-    </gazebo>
-    <gazebo reference="front_right_wheel">
-        <material>${wheels_color}</material>
-        <mu1>0.001</mu1>
-        <mu2>0.001</mu2>
-    </gazebo>
+<robot name="ugv"
+	xmlns:xacro="http://www.ros.org/wiki/xacro">
+	<gazebo reference="base_link">
+		<!-- <material>
+			<ambient>1 0 0 1</ambient>
+			<diffuse>1 0 0 1</diffuse>
+			<specular>0.1 0.1 0.1 1</specular>
+		</material> -->
+	</gazebo>
+	<gazebo reference="front_left_wheel">
+		<!-- <material>
+			<ambient>1 0 0 1</ambient>
+			<diffuse>1 0 0 1</diffuse>
+			<specular>0.1 0.1 0.1 1</specular>
+		</material> -->
+		<mu1>0.001</mu1>
+		<mu2>0.001</mu2>
+	</gazebo>
+	<gazebo reference="rear_left_wheel">
+		<!-- <material>
+			<ambient>1 0 0 1</ambient>
+			<diffuse>1 0 0 1</diffuse>
+			<specular>0.1 0.1 0.1 1</specular>
+		</material> -->
+		<mu1>0.001</mu1>
+		<mu2>0.001</mu2>
+	</gazebo>
+	<gazebo reference="rear_right_wheel">
+		<!-- <material>
+			<ambient>1 0 0 1</ambient>
+			<diffuse>1 0 0 1</diffuse>
+			<specular>0.1 0.1 0.1 1</specular>
+		</material> -->
+		<mu1>0.001</mu1>
+		<mu2>0.001</mu2>
+	</gazebo>
+	<gazebo reference="front_right_wheel">
+		<!-- <material>
+			<ambient>1 0 0 1</ambient>
+			<diffuse>1 0 0 1</diffuse>
+			<specular>0.1 0.1 0.1 1</specular>
+		</material> -->
+		<mu1>0.001</mu1>
+		<mu2>0.001</mu2>
+	</gazebo>
 </robot>

File: ugv_description/gazebo/lidar.xacro (robot description, xacro)
@@ -1,35 +1,41 @@
 <?xml version="1.0" encoding="UTF-8"?>
 <robot>
-    <gazebo reference="lidar_link">
-        <material>Gazebo/Black</material>
-        <mu1>0.2</mu1>
-        <mu2>0.2</mu2>
-        <self_collide>true</self_collide>
-        <sensor name="laser" type="ray">
-            <pose>0 0 0 0 0 0</pose>
-            <visualize>true</visualize>
-            <update_rate>10</update_rate>
-            <always_on>1</always_on>
-            <ray>
-                <scan>
-                    <horizontal>
-                        <samples>360</samples>
-                        <min_angle>-3.14</min_angle>
-                        <max_angle>3.14</max_angle>
-                    </horizontal>
-                </scan>
-                <range>
-                    <min>0.3</min>
-                    <max>12</max>
-                </range>
-            </ray>
-            <plugin name="laser_controller" filename="libgazebo_ros_ray_sensor.so">
-                <ros>
-                    <remapping>~/out:=scan</remapping>
-                </ros>
-                <output_type>sensor_msgs/LaserScan</output_type>
-                <frame_name>lidar_link</frame_name>
-            </plugin>
+    <gazebo>
+        <plugin filename="gz-sim-sensors-system" name="gz::sim::systems::Sensors">
+          <render_engine>ogre2</render_engine>
+        </plugin>
+      </gazebo>
+      <gazebo reference="lidar_link" >
+        <sensor name="lidar_link" type="gpu_lidar">
+          <gz_frame_id>lidar_link</gz_frame_id>
+          <topic>scan</topic>
+          <update_rate>30</update_rate>
+          <visualize>true</visualize>
+          <always_on>true</always_on>
+          <lidar>
+            <scan>
+              <horizontal>
+                <samples>2800</samples>
+                <resolution>1</resolution>
+                <min_angle>-3.14</min_angle>
+                <max_angle>3.14</max_angle>
+              </horizontal>
+              <vertical>
+                <samples>1</samples>
+                <resolution>0.1</resolution>
+                <min_angle>0.0</min_angle>
+                <max_angle>0.0</max_angle>
+              </vertical>
+            </scan>
+            <range>
+              <min>0.2</min>
+              <max>30.0</max>
+              <resolution>0.01</resolution>
+            </range>
+            <frame_id>/lidar_head_link</frame_id>
+          </lidar>
+          <alwaysOn>ture</alwaysOn>
+          <visualize>true</visualize>
         </sensor>
-    </gazebo>
+      </gazebo>
 </robot>

File: ugv_description/urdf/ugv.macro.xacro (robot description, xacro)
@@ -4,5 +4,5 @@
         <xacro:include filename="$(find ugv_description)/urdf/ugv_core.xacro"/>
         <xacro:if value="$(arg is_sim)">
-            <xacro:include filename="$(find ugv_description)/gazebo/gazebo.xacro"/>
+            <!-- <xacro:include filename="$(find ugv_description)/gazebo/gazebo.xacro"/> -->
             <xacro:include filename="$(find ugv_description)/gazebo/lidar.xacro"/>
             <!--        <xacro:include filename="gazebo/imu.xacro"/>-->
